File: rpi_ad7705-2.brd (EAGLE design)
At the start: 81.3 x 54.3 mm, 26 parts, among them IC1 ULN2003AN

Commit message: Added files via upload
Update these two files for value changes
Parts:
- R1: value 22K -> 22
- R3: value 13 -> 10K
- R4: value 62 -> 10K
Changed lines of the file:
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@@
 </element>
 <element name="C2" library="capacitor-wima" package="C5B2.5" value="0.1uF" x="8.255" y="33.02"/>
-<element name="R1" library="resistor" package="0207/10" value="22K" x="21.59" y="13.97" rot="R90"/>
+<element name="R1" library="resistor" package="0207/10" value="22" x="21.59" y="13.97" rot="R90"/>
 <element name="SV4" library="con-lstb" package="MA04-1" value="GPIO" x="53.975" y="41.91" rot="R90">
 <attribute name="MF" value="" x="53.975" y="41.91" size="1.778" layer="27" rot="R90" display="off"/>
@@
 <element name="C4" library="capacitor-wima" package="C5B2.5" value="0.1uF" x="25.4" y="15.875" rot="R90"/>
 <element name="C5" library="rcl" package="TT2D7" value="1uF/tantalum" x="31.75" y="15.875" rot="R270"/>
-<element name="R3" library="resistor" package="0207/10" value="13" x="48.26" y="11.43" rot="R90"/>
-<element name="R4" library="resistor" package="0207/10" value="62" x="56.515" y="11.43" rot="R270"/>
+<element name="R3" library="resistor" package="0207/10" value="10K" x="48.26" y="11.43" rot="R90"/>
+<element name="R4" library="resistor" package="0207/10" value="10K" x="56.515" y="11.43" rot="R270"/>
 <element name="IC1" library="uln-udn" package="DIL16" value="ULN2003AN" x="53.34" y="26.035"/>
 <element name="LED1" library="led" package="LED3MM" value="TLLG4400" x="74.93" y="46.99" rot="R270">
